File: board/6-dc34-moth-badge-attiny.kicad_sch (KiCad schematic)
At the start: 13 parts, among them SW3 Mode SW, SW4 ATtiny battery power, U2 ATtiny814-SS

Commit message: v1.0 board
Connections:
- net GPIO 2: now reaches U2.13 (PA3)
- net GPIO 1: now reaches U2.3 (PA5)
- no-connect marks 3 -> 1
Changed lines of the file:
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@@
-	)
-	(no_connect
-		(at 139.7 85.09)
 	)
 	(no_connect
 		(at 153.67 59.69)
 	)
-	(no_connect
-		(at 139.7 90.17)
-	)
 	(wire
 		(pts
@@
 	(wire
 		(pts
+			(xy 139.7 90.17) (xy 144.78 90.17)
+		)
+		(stroke
+			(width 0)
+			(type default)
+		)
+	)
+	(wire
+		(pts
 			(xy 139.7 82.55) (xy 144.78 82.55)
 		)
@@
 		(pts
 			(xy 139.7 80.01) (xy 144.78 80.01)
+		)
+		(stroke
+			(width 0)
+			(type default)
+		)
+	)
+	(wire
+		(pts
+			(xy 139.7 85.09) (xy 144.78 85.09)
 		)
 		(stroke
@@
 		(effects
 			(font
+				(size 1.27 1.27)
+			)
+			(justify left)
+		)
+	)
+	(hierarchical_label "GPIO 2"
+		(shape bidirectional)
+		(at 144.78 85.09 0)
+		(effects
+			(font
+				(size 1.27 1.27)
+			)
+			(justify left)
+		)
+	)
+	(hierarchical_label "GPIO 1"
+		(shape bidirectional)
+		(at 144.78 90.17 0)
+		(effects
+			(font
