File: board/6-dc34-moth-badge.kicad_sch (KiCad schematic)
At the start: 23 parts, among them J1 USB C, J2 USB Tongue, J3 External UPDI, SW1 SW_SPDT, SW2 SW_SPDT, U1 CH340E, U3 AP2112K-3.3, X1 Simple_Addon_v2

Commit message: board v0.1
Parts:
- removed J3: External UPDI, Connector_PinHeader_2.54mm:PinHeader_1x03_P2.54mm_Vertical, symbol Connector_Generic:Conn_01x03
- added J3: Conn_01x08, Connector_PinHeader_2.54mm:PinHeader_1x08_P2.54mm_Vertical, symbol Connector_Generic:Conn_01x08
- added R13: 470, Resistor_SMD:R_1206_3216Metric_Pad1.30x1.75mm_HandSolder, symbol Device:R
- C1, C2: footprint (none) -> Capacitor_SMD:C_1206_3216Metric_Pad1.33x1.80mm_HandSolder
- D1, D2: footprint (none) -> LED_SMD:LED_1206_3216Metric_Pad1.42x1.75mm_HandSolder
- D3, D4, D5, D6, D7: footprint (none) -> Diode_SMD:D_1206_3216Metric_Pad1.42x1.75mm_HandSolder
- J1: footprint (none) -> USB4216-03-A:USB421603A
- J2: footprint (none) -> USB_LepiLabs:USB_Tongue
- R1, R11, R12, R2, R3: footprint (none) -> Resistor_SMD:R_1206_3216Metric_Pad1.30x1.75mm_HandSolder
- R4: value R -> 470; footprint (none) -> Resistor_SMD:R_1206_3216Metric_Pad1.30x1.75mm_HandSolder
- SW1, SW2: footprint (none) -> SLW-88229-2-SMT-TR:SLW882292SMTTR
- X1: footprint (none) -> Simple_Addon_v2:Simple_Addon_v2-SAO-2x3
Connections:
- net +3.3V: now also R13.1; no longer D1.2 (A)
- net External UPDI: now also J3.6 (Pin_6)
- net GND: now also J3.8 (Pin_8)
- net PWR select: now also J3.7 (Pin_7)
- new net: D1.2 (A), R13.2
- no-connect marks 6 -> 11
