File: board/6-dc34-moth-badge.kicad_sch (KiCad schematic)
At the start: 24 parts, among them J1 USB C, J2 USB Tongue, J3 Conn_01x08, SW1 SW_SPDT, SW2 SW_SPDT, U1 CH340E, U3 AP2112K-3.3, X1 Simple_Addon_v2

Commit message: v1.0 board
Parts:
- added C3, C4: 0.1u, Capacitor_SMD:C_1206_3216Metric_Pad1.33x1.80mm_HandSolder, symbol Device:C_Small
- added F1: 1A, Fuse:Fuse_1206_3216Metric_Pad1.42x1.75mm_HandSolder, symbol Device:Fuse_Small
Connections:
- net +5V: no longer U1.7 (VCC)
- net GND: now also C3.2, C4.2
- net PWR select: now also U1.7 (VCC), C4.1
- net at D5.2 (A): now also F1.2; no longer J2.1 (VBUS)
- net GPIO 1: now reaches X1.5 (GPIO1)
- net GPIO 2: now reaches X1.6 (GPIO2)
- net at U1.10 (V3): now also C3.1
- new net: F1.1, J2.1 (VBUS)
- no-connect marks 11 -> 8
Other:
- sheet ATtiny ports: added GPIO 1, GPIO 2; removed none
- moved on the sheet: D5, R11, R12

Commit message: fix CG on switches
Parts:
- SW1, SW2: symbol Switch:SW_SPDT -> Switch:SW_SPDT_312
Connections:
- net +3.3V: now also SW2.2 (C); no longer SW2.1 (A)
- net ATtiny UPDI: now also SW1.2 (C); no longer SW1.1 (A)
- net PWR select: now also SW2.1 (B); no longer SW2.2 (B)
- net at R4.2: now also SW1.1 (B); no longer SW1.2 (B)
