File: board/6-dc34-moth-badge.kicad_pcb (KiCad board)
At the start: 2 copper layers, 75.9 x 96.4 mm, 41 parts, among them J1 USB C, J2 USB Tongue, J3 Conn_01x08, SW1 SW_SPDT, SW2 SW_SPDT, SW3 Mode SW, SW4 ATtiny battery power, U1 CH340E, U2 ATtiny814-SS, U3 AP2112K-3.3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

Commit message: updates
Routing:
- net /USB D+: track 21.8 -> 33.9 mm
- net /USB D-: track 21.8 -> 33.2 mm
- net Net-(D5-A): track 17.7 -> 21.3 mm
- net GND: vias 4 -> 20
