File: board/6-dc34-moth-badge.kicad_pcb (KiCad board)
At the start: 2 copper layers, 75.9 x 96.4 mm, 41 parts, among them J1 USB C, J2 USB Tongue, J3 Conn_01x08, SW1 SW_SPDT, SW2 SW_SPDT, SW3 Mode SW, SW4 ATtiny battery power, U1 CH340E, U2 ATtiny814-SS, U3 AP2112K-3.3, X1 Simple_Addon_v2

Commit message: v1.0 board
Parts:
- added C3: 0.1u, Capacitor_SMD:C_1206_3216Metric_Pad1.33x1.80mm_HandSolder, B.Cu at (136.5, 130.8)
- added C4: 0.1u, Capacitor_SMD:C_1206_3216Metric_Pad1.33x1.80mm_HandSolder, B.Cu at (129.2, 125.2)
- added F1: 1A, Fuse:Fuse_1206_3216Metric_Pad1.42x1.75mm_HandSolder, B.Cu at (141.3, 115.2)
- moved D6 12.9 mm to (134.0, 111.2), turned to 0 degrees
- moved D5 6.84 mm to (147.0, 115.2), turned to 180 degrees
- moved D3 6.45 mm to (132.2, 130.8), turned to -90 degrees
- moved R2 4.75 mm to (136.0, 135.8)
- moved R4 3.63 mm to (133.9, 107.5)
- moved C1 1.78 mm to (134.1, 118.8)
- moved C2 1.78 mm to (134.1, 115.3), turned to 0 degrees
- moved U3 1.78 mm to (133.6, 123.5)
- moved R1 1.45 mm to (156.0, 138.2)
- moved D7 1.23 mm to (140.8, 110.0)
Connections:
- J2 pad 1: Net-(D5-A) -> Net-(J2-VBUS)
- U1 pad 10: unconnected-(U1-V3-Pad10) -> Net-(U1-V3)
- U1 pad 7: +5V -> /PWR select
- U2 pad 13: unconnected-(U2-PA3-Pad13) -> /GPIO 2
- U2 pad 3: unconnected-(U2-PA5-Pad3) -> /GPIO 1
- X1 pad 5: unconnected-(X1-GPIO1-Pad5) -> /GPIO 1
- X1 pad 6: unconnected-(X1-GPIO2-Pad6) -> /GPIO 2
Routing:
- net /PWR select: track 72.5 -> 110.7 mm
- net /GPIO 2: track 0.00 -> 27.4 mm
- net Net-(J2-VBUS): track 0.00 -> 24.5 mm
- net /GPIO 1: track 0.00 -> 22.8 mm
- net Net-(D5-A): track 21.3 -> 6.74 mm
- net Net-(D6-K): track 13.3 -> 25.7 mm
- net Net-(U1-V3): track 0.00 -> 10.2 mm, vias 0 -> 2
- net Net-(D3-A): track 14.8 -> 23.1 mm
- net +5V: track 72.1 -> 64.2 mm, vias 2 -> 4
- net +3.3V: track 161.1 -> 165.7 mm
- net Net-(D6-A): track 31.4 -> 27.5 mm
- net GND: track 5.13 -> 7.52 mm, vias 20 -> 27
- net Net-(J1-CC2): track 10.5 -> 8.25 mm
- net Net-(D7-A): track 15.9 -> 18.0 mm, vias 0 -> 2
- net Net-(J1-CC1): track 8.81 -> 9.81 mm
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Other:
- board text added: "1A MAX"
- board text added: "CR2032"
- board text added: "GND +V UPDI"
- board text added: "Mode"
- board text added: "PA4"
- board text added: "PA7 PB3 PB2"
- board text added: "PB0 PA6 PB1"
- board text added: "R G B"
- board text added: "v1.0"
- board text removed: "v0.1"
