File: tongue_fpc/6-dc34-moth-badge-tongue.kicad_pcb (KiCad board)
At the start: 2 copper layers, 142.4 x 12 mm, 2 parts, among them J1 USB_A, J2 Conn_01x04

Commit message: updates
Parts:
- J1: moved to F.Cu
- turned J2 to -90 degrees
Connections:
- J2 pad 1: GND -> /VCC
- J2 pad 4: /VCC -> GND
Routing:
- net GND: track 150.1 -> 0.00 mm, vias 1 -> 9
- net /VCC: track 150.1 -> 153.0 mm, vias 1 -> 2
- net /D-: track 150.9 -> 150.7 mm, vias 1 -> 0
- net /D+: track 150.9 -> 150.7 mm, vias 1 -> 0
