File: tongue_fpc/6-dc34-moth-badge-tongue.kicad_sch (KiCad schematic)
At the start: 2 parts, among them J1 USB_A, J2 Conn_01x04

Commit message: updates
Connections:
- net GND: now also J2.4 (Pin_4); no longer J2.1 (Pin_1)
- net VCC: now also J2.1 (Pin_1); no longer J2.4 (Pin_4)
Changed lines of the file:
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@@
 	(wire
 		(pts
-			(xy 162.56 101.6) (xy 171.45 101.6)
+			(xy 168.91 101.6) (xy 171.45 101.6)
 		)
 		(stroke
@@
 	)
 	(label "VCC"
-		(at 168.91 109.22 180)
+		(at 168.91 101.6 180)
 		(effects
 			(font
@@
 		)
 	)
+	(label "D-"
+		(at 168.91 106.68 180)
+		(effects
+			(font
+				(size 1.27 1.27)
+			)
+			(justify right bottom)
+		)
+	)
 	(label "D+"
 		(at 168.91 104.14 180)
-		(effects
-			(font
-				(size 1.27 1.27)
-			)
-			(justify right bottom)
-		)
-	)
-	(label "D-"
-		(at 168.91 106.68 180)
 		(effects
 			(font
@@
 	(symbol
 		(lib_id "power:GND")
-		(at 162.56 101.6 0)
+		(at 168.91 109.22 0)
 		(unit 1)
 		(body_style 1)
@@
 		(fields_autoplaced yes)
 		(property "Reference" "#PWR02"
-			(at 162.56 107.95 0)
+			(at 168.91 115.57 0)
 			(hide yes)
 			(show_name no)
@@
 		)
 		(property "Value" "GND"
-			(at 162.56 106.68 0)
+			(at 168.91 114.3 0)
 			(show_name no)
 			(do_not_autoplace no)
@@
 		)
 		(property "Footprint" ""
-			(at 162.56 101.6 0)
+			(at 168.91 109.22 0)
 			(hide yes)
 			(show_name no)
@@
 		)
 		(property "Datasheet" ""
-			(at 162.56 101.6 0)
+			(at 168.91 109.22 0)
 			(hide yes)
 			(show_name no)
@@
 		)
 		(property "Description" "Power symbol creates a global label with name \"GND\" , ground"
-			(at 162.56 101.6 0)
-			(hide yes)
-			(show_name no)
+			(at 168.91 109.22 0)
+			(hide yes)
+			(show_name no)
